Commit message: Added gazebo simulation

File: robotiq_description/urdf/robotiq_hande_gripper.transmission.xacro (robot description, xacro)
@@ -5,5 +5,5 @@
       <type>transmission_interface/SimpleTransmission</type>
       <joint name="${prefix}hande_left_finger_joint">
-        <hardwareInterface>hardware_interface/PositionJointInterface</hardwareInterface>
+        <hardwareInterface>hardware_interface/EffortJointInterface</hardwareInterface>
       </joint>
       <actuator name="${prefix}hande_left_finger_motor">
@@ -11,15 +11,15 @@
       </actuator>
     </transmission>
-    <!-- <transmission name="${prefix}hande_right_finger_trans">
+    <transmission name="${prefix}hande_right_finger_trans">
       <type>transmission_interface/SimpleTransmission</type>
       <joint name="${prefix}hande_right_finger_joint">
-        <hardwareInterface>hardware_interface/PositionJointInterface</hardwareInterface>
+        <hardwareInterface>hardware_interface/EffortJointInterface</hardwareInterface>
       </joint>
       <actuator name="${prefix}hande_right_finger_motor">
         <mechanicalReduction>1</mechanicalReduction>
       </actuator>
-    </transmission> -->
+    </transmission>
     <!-- Mimic joints -->
-    <gazebo>
+    <!-- <gazebo>
       <plugin filename="libgazebo_mimic_joint_plugin.so" name="${prefix}mimic_robotiq_hande">
         <joint>${prefix}hande_left_finger_joint</joint>
@@ -28,5 +28,5 @@
         <offset>0.0</offset>
       </plugin>
-    </gazebo>
+    </gazebo> -->
   </xacro:macro>
 </robot>

File: robotiq_description/urdf/robotiq_hande_gripper.urdf.xacro (robot description, xacro)
@@ -99,21 +99,21 @@
       <axis xyz="1 0 0"/>
       <limit effort="130" lower="0" upper="0.025" velocity="0.15"/>
-      <mimic joint="${prefix}hande_left_finger_joint" multiplier="1" offset="0"/>
+      <!-- <mimic joint="${prefix}hande_left_finger_joint" multiplier="1" offset="0"/> -->
     </joint>
-      <!-- Improve grasping physics -->
-      <gazebo reference="${prefix}hande_left_finger">
-        <kp>1000000.0</kp>
-        <kd>1.0</kd>
-        <mu1>1.0</mu1>
-        <mu2>1.0</mu2>
-        <minDepth>0.001</minDepth>
-      </gazebo>
-      <gazebo reference="${prefix}hande_right_finger">
-        <kp>1000000.0</kp>
-        <kd>1.0</kd>
-        <mu1>1.0</mu1>
-        <mu2>1.0</mu2>
-        <minDepth>0.001</minDepth>
-      </gazebo>
+    <!-- Improve grasping physics -->
+    <gazebo reference="${prefix}hande_left_finger">
+      <kp>1000000.0</kp>
+      <kd>1.0</kd>
+      <mu1>1.0</mu1>
+      <mu2>1.0</mu2>
+      <minDepth>0.001</minDepth>
+    </gazebo>
+    <gazebo reference="${prefix}hande_right_finger">
+      <kp>1000000.0</kp>
+      <kd>1.0</kd>
+      <mu1>1.0</mu1>
+      <mu2>1.0</mu2>
+      <minDepth>0.001</minDepth>
+    </gazebo>
     <xacro:robotiq_hande_gripper_transmission prefix="${prefix}" />
   </xacro:macro>
