Commit message: marco : added param to run ros control gazebo

File: robotiq_gazebo/robotiq_gazebo/urdf/gripper_gazebo.xacro (robot description, xacro)
@@ -1,5 +1,5 @@
 <?xml version="1.0"?>
 <robot xmlns:xacro="http://ros.org/wiki/xacro" name="robotiq">
-  <xacro:macro name="robotiq_gazebo" params="prefix parent *origin">
+  <xacro:macro name="robotiq_gazebo" params="prefix parent *origin launch_gazebo_ros_control_plugin='yes'">
     <!-- includes -->
     <xacro:include filename="$(find robotiq_description)/urdf/robotiq_hande_gripper.urdf.xacro" />
@@ -10,10 +10,12 @@
     </xacro:robotiq_hande_gripper>
     <!-- Loading Gazebo plugins -->
-    <gazebo>
-      <plugin name="ros_control" filename="libgazebo_ros_control.so">
-        <!--robotNamespace>/</robotNamespace-->
-        <!--robotSimType>gazebo_ros_control/DefaultRobotHWSim</robotSimType-->
-      </plugin>
-    </gazebo>
+    <xacro:if value="${launch_gazebo_ros_control_plugin == 'yes'}">
+      <gazebo>
+        <plugin name="ros_control" filename="libgazebo_ros_control.so">
+          <!--robotNamespace>/</robotNamespace-->
+          <!--robotSimType>gazebo_ros_control/DefaultRobotHWSim</robotSimType-->
+        </plugin>
+      </gazebo>
+    </xacro:if>
     <!-- Disabling gravity -->
     <gazebo reference="hande_left_finger">

Commit message: marco : changed yes/no to true/false

File: robotiq_gazebo/robotiq_gazebo/urdf/gripper_gazebo.xacro (robot description, xacro)
@@ -1,5 +1,5 @@
 <?xml version="1.0"?>
 <robot xmlns:xacro="http://ros.org/wiki/xacro" name="robotiq">
-  <xacro:macro name="robotiq_gazebo" params="prefix parent *origin launch_gazebo_ros_control_plugin='yes'">
+  <xacro:macro name="robotiq_gazebo" params="prefix parent *origin launch_gazebo_ros_control_plugin='true'">
     <!-- includes -->
     <xacro:include filename="$(find robotiq_description)/urdf/robotiq_hande_gripper.urdf.xacro" />
@@ -10,5 +10,5 @@
     </xacro:robotiq_hande_gripper>
     <!-- Loading Gazebo plugins -->
-    <xacro:if value="${launch_gazebo_ros_control_plugin == 'yes'}">
+    <xacro:if value="${launch_gazebo_ros_control_plugin}">
       <gazebo>
         <plugin name="ros_control" filename="libgazebo_ros_control.so">
